File: kicad/connectivity.kicad_sch (KiCad schematic)
At the start: 0 parts

Commit message: Very messy checkpointing post filling of system disk.
Parts:
- added U5: nRF52832-QFxx, Package_DFN_QFN:QFN-48-1EP_6x6mm_P0.4mm_EP4.6x4.6mm, symbol MCU_Nordic:nRF52832-QFxx
Connections:
- new net: U5.13 (VDD), U5.36 (VDD), U5.48 (VDD)
- new net: U5.31 (VSS), U5.45 (VSS), U5.49 (VSS)
Other:
- company: iGrow UG -> Kiwi Devices Limited
- title: (none) -> Connectivity
Changed lines of the file:
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@@
-(kicad_sch (version 20201015) (generator eeschema)
-  (paper "A4")
-  (title_block
-    (company "iGrow UG")
-  )
+(kicad_sch
+	(version 20240417)
+	(generator "eeschema")
+	(generator_version "8.99")
+	(paper "A4")
+	(title_block
+		(title "Connectivity")
+		(date "2024-05-09")
+		(company "Kiwi Devices Limited")
+	)
+	(symbol
+		(lib_id "MCU_Nordic:nRF52832-QFxx")
+		(at 134.62 91.44 0)
+		(unit 1)
+		(exclude_from_sim no)
+		(in_bom yes)
+		(on_board yes)
+		(dnp no)
+		(fields_autoplaced yes)
+		(property "Reference" "U5"
+			(at 136.8141 134.62 0)
+			(effects
+				(font
+					(size 1.27 1.27)
+				)
+				(justify left)
+			)
+		)
+		(property "Value" "nRF52832-QFxx"
+			(at 136.8141 137.16 0)
+			(effects
+				(font
+					(size 1.27 1.27)
+				)
+				(justify left)
+			)
+		)
+		(property "Footprint" "Package_DFN_QFN:QFN-48-1EP_6x6mm_P0.4mm_EP4.6x4.6mm"
+			(at 134.62 144.78 0)
+			(effects
+				(font
+					(size 1.27 1.27)
+				)
+				(hide yes)
+			)
+		)
+		(property "Datasheet" "http://infocenter.nordicsemi.com/pdf/nRF52832_PS_v1.4.pdf"
+			(at 121.92 86.36 0)
+			(effects
+				(font
+					(size 1.27 1.27)
+				)
+				(hide yes)
+			)
+		)
+		(property "Description" "Multiprotocol BLE/2.4GHz Cortex-M4 SoC, QFN-48"
+			(at 134.62 91.44 0)
+			(effects
+				(font
+					(size 1.27 1.27)
+				)
+				(hide yes)
+			)
+		)
+		(pin "31"
+		)
+		(pin "2"
+		)
+		(pin "36"
+		)
+		(pin "17"
+		)
+		(pin "3"
+		)
+		(pin "6"
+		)
+		(pin "48"
+		)
+		(pin "42"
+		)
+		(pin "38"
+		)
+		(pin "44"
+		)
+		(pin "47"
+		)
+		(pin "16"
+		)
+		(pin "45"
+		)
+		(pin "14"
+		)
+		(pin "49"
+		)
+		(pin "1"
+		)
+		(pin "20"
+		)
+		(pin "35"
+		)
+		(pin "22"
+		)
+		(pin "26"
+		)
+		(pin "28"
+		)
+		(pin "21"
+		)
+		(pin "34"
+		)
+		(pin "25"
+		)
+		(pin "19"
+		)
+		(pin "23"
+		)
+		(pin "12"
+		)
+		(pin "5"
+		)
+		(pin "41"
+		)
+		(pin "32"
+		)
+		(pin "8"
+		)
+		(pin "33"
+		)
+		(pin "9"
+		)
+		(pin "4"
+		)
+		(pin "27"
+		)
+		(pin "13"
+		)
+		(pin "46"
+		)
+		(pin "29"
+		)
+		(pin "7"
+		)
+		(pin "18"
+		)
+		(pin "11"
+		)
+		(pin "43"
+		)
+		(pin "30"
+		)
+		(pin "40"
+		)
+		(pin "37"
+		)
+		(pin "24"
+		)
+		(pin "39"
+		)
+		(pin "10"
+		)
+		(pin "15"
+		)
+		(instances
+			(project "led-supply"
+				(path "/a5bc576a-16b1-469b-95bf-cd73ad37d133/f1c533f3-880e-43af-939d-d1b04b8807dd"
+					(reference "U5")
+					(unit 1)
+				)
+			)
+		)
+	)
 )
