File: kicad/led-string.kicad_sch (KiCad schematic)
At the start: 15 parts

Commit message: Very messy checkpointing post filling of system disk.
Parts:
- D1, D10, D11, D12, D13, D14, D15, D2, D3, D4, D5, D6, D7, D8, D9: footprint (none) -> led-supply:SPMWHD32AMH5XAV5SK
Other:
- company: iGrow UG -> Kiwi Devices Limited
