File: kicad/led-supply.kicad_sch (KiCad schematic)
At the start: 0 parts

Commit message: Very messy checkpointing post filling of system disk.
Other:
- added sheet Line Protection (line-protection.kicad_sch)
- company: iGrow UG -> Kiwi Devices Limited
