File: kicad/rectifier-control.kicad_sch (KiCad schematic)
At the start: 0 parts

Commit message: Very messy checkpointing post filling of system disk.
Parts:
- added C10, C11, C12, C13, C14, C16, C17, C9: 100n, symbol Device:C
- added C15: 1u, symbol Device:C
- added D20: ESDA6V1SC5, Package_TO_SOT_SMD:SOT-23-5, symbol Power_Protection:ESDA6V1SC5
- added FB1, FB2: 300R @ 100MHz, symbol Device:FerriteBead
- added FB3: 600R @ 100MHz, symbol Device:FerriteBead
- added J1: Conn_ARM_SWD_TagConnect_TC2030, Connector:Tag-Connect_TC2030-IDC-FP_2x03_P1.27mm_Vertical, symbol Connector:Conn_ARM_SWD_TagConnect_TC2030
- added JP1, JP2: SolderJumper_2_Open, symbol Jumper:SolderJumper_2_Open
- added U4: STM32G474RETx, Package_QFP:LQFP-64_10x10mm_P0.5mm, symbol MCU_ST_STM32G4:STM32G474RETx
Connections:
- new net: C17.1, FB1.1, JP2.2 (B)
- new net +3V3: J1.1 (VCC)
- new net GNDA: C17.2, U4.27 (VSSA)
- new net GNDD: C10.2, C11.2, C12.2, C13.2, C16.2, C9.2, D20.2 (A), FB3.2, J1.5 (GND), JP1.2 (B), U4.15 (VSS), U4.31 (VSS), U4.47 (VSS), U4.63 (VSS)
- new net NRST: D20.5 (K), J1.3 (~{RESET}), U4.7 (PG10)
- new net SWCLK: D20.4 (K), J1.4 (SWCLK), U4.50 (PA14)
- new net SWDIO: D20.3 (K), J1.2 (SWDIO), U4.49 (PA13)
- new net SWO: D20.1 (K), J1.6 (SWO), U4.56 (PB3)
- new net VDD: C10.1, C11.1, C12.1, C13.1, C9.1, FB2.2, U4.16 (VDD), U4.32 (VDD), U4.48 (VDD), U4.64 (VDD)
- new net VDDA: C14.1, C15.1, FB2.1, U4.29 (VDDA)
- new net VREF: JP2.1 (A)
- new net VREFP: FB1.2, U4.28 (VREF+)
- new net VSSA: C14.2, C15.2, C16.1, FB3.1, JP1.1 (A)
Other:
- company: iGrow UG -> Kiwi Devices Limited
- title: (none) -> Rectifier Control
