File: kicad/rectifier.kicad_sch (KiCad schematic)
At the start: 0 parts

Commit message: Very messy checkpointing post filling of system disk.
Parts:
- added C18: C_Polarized, symbol Device:C_Polarized
- added D21: GBU8J, Diode_THT:Diode_Bridge_Vishay_GBU, symbol Diode_Bridge:GBU8J
- added L1: L_Ferrite, symbol Device:L_Ferrite
- added Q1: BC807, Package_TO_SOT_SMD:SOT-23, symbol Transistor_BJT:BC807
- added Q2: BC817, Package_TO_SOT_SMD:SOT-23, symbol Transistor_BJT:BC817
- added Q3, Q5: IPDD60R190G7, Package_TO_SOT_SMD:Infineon_PG-HDSOP-10-1, symbol Transistor_FET:IPDD60R190G7
- added Q4: 2N7002, Package_TO_SOT_SMD:SOT-23, symbol Transistor_FET:2N7002
- added R1, R2, R3: R, symbol Device:R
Connections:
- new net: C18.1, Q5.10 (D), Q5.6 (D), Q5.7 (D), Q5.8 (D), Q5.9 (D)
- new net: Q1.1 (B), Q2.1 (B), R3.2
- new net: Q1.2 (E), Q2.3 (C), R1.1
- new net: Q3.1 (G), R1.2
- new net: L1.2, Q3.10 (D), Q3.6 (D), Q3.7 (D), Q3.8 (D), Q3.9 (D), Q5.2 (DS), Q5.3 (PS), Q5.4 (PS), Q5.5 (PS)
- new net: Q4.3 (D), R2.1, R3.1
- new net: D21.1 (+), L1.1
- new net +12V: Q1.3 (C), R2.2
- new net GATE_DRIVE_1: Q4.1 (G)
- new net GND: C18.2, D21.4 (-), Q3.2 (DS), Q3.3 (PS), Q3.4 (PS), Q3.5 (PS)
- new net GNDD: Q2.2 (E), Q4.2 (S)
- new net L_COND: D21.3
- new net N_COND: D21.2
Other:
- company: iGrow UG -> Kiwi Devices Limited
